Commit message: fix(config): update counts_per_rev, add velocity controller gains, add joint limits to urdf

File: urdf/robot.urdf (robot description, URDF)
Before this commit: robot canopen_robot, 7 links, 6 joints
Joints:
- joint joint_1: limit (none) -> lower=-31.416 upper=31.416 effort=100 velocity=3.14; type continuous -> revolute
- joint joint_2: limit (none) -> lower=-31.416 upper=31.416 effort=100 velocity=3.14; type continuous -> revolute
- joint joint_3: limit (none) -> lower=-31.416 upper=31.416 effort=100 velocity=3.14; type continuous -> revolute
- joint joint_4: limit (none) -> lower=-31.416 upper=31.416 effort=100 velocity=3.14; type continuous -> revolute
- joint joint_5: limit (none) -> lower=-31.416 upper=31.416 effort=100 velocity=3.14; type continuous -> revolute
- joint joint_6: limit (none) -> lower=-31.416 upper=31.416 effort=100 velocity=3.14; type continuous -> revolute

Commit message: fix(Eyou_Canopen_Master): align runtime joint names with car_urdf

File: urdf/robot.urdf (robot description, URDF)
Before this commit: robot canopen_robot, 7 links, 6 joints
Joints:
- removed joint joint_1
- removed joint joint_2
- removed joint joint_3
- removed joint joint_4
- removed joint joint_5
- removed joint joint_6
- added joint elbow_pitch_joint: type revolute, parent joint_2_link, child joint_3_link, axis 0 0 1, limit lower=-31.416 upper=31.416 effort=100 velocity=3.14
- added joint shoulder_pitch_joint: type revolute, parent joint_1_link, child joint_2_link, axis 0 0 1, limit lower=-31.416 upper=31.416 effort=100 velocity=3.14
- added joint shoulder_yaw_joint: type revolute, parent base_link, child joint_1_link, axis 0 0 1, limit lower=-31.416 upper=31.416 effort=100 velocity=3.14
- added joint wrist_pitch_joint: type revolute, parent joint_3_link, child joint_4_link, axis 0 0 1, limit lower=-31.416 upper=31.416 effort=100 velocity=3.14
- added joint wrist_roll_joint: type revolute, parent joint_4_link, child joint_5_link, axis 0 0 1, limit lower=-31.416 upper=31.416 effort=100 velocity=3.14
- added joint wrist_yaw_joint: type revolute, parent joint_5_link, child joint_6_link, axis 0 0 1, limit lower=-31.416 upper=31.416 effort=100 velocity=3.14
